Commit message: attach camera to M0609

File: dsr_description2/xacro/macro.m0609.white.xacro (robot description, xacro)
@@ -243,4 +243,121 @@
 			</visual>
 		</link>
+		<!-- end effector axis for visualization-->
+		<link name="link_6_z_rod">
+			<visual>
+				<origin rpy="0 0 0" xyz="0 0 0" />
+				<geometry>
+					<cylinder radius="0.005" length="0.5" /> </geometry>
+				<material name="blue">
+					<color rgba="0.0 0.0 1.0 1.0" />
+				</material>
+			</visual>
+			<inertial>
+				<mass value="1e-5" />
+				<origin xyz="0 0 0" rpy="0 0 0" />
+				<inertia ixx="1e-6" ixy="0" ixz="0" iyy="1e-6" iyz="0" izz="1e-6" />
+			</inertial>
+		</link>
+		<joint name="link_6_z_rod_joint" type="fixed">
+			<parent link="link_6" />
+			<child link="link_6_z_rod" />
+			<origin xyz="0 0 0" rpy="0 0 0" />
+		</joint>
+		<gazebo reference="link_6_z_rod">
+			<visual>
+				<material>
+					<ambient>1 0 0 1</ambient>
+					<diffuse>1 0 0 1</diffuse>
+					<specular>0.1 0.1 0.1 1</specular>
+				</material>
+			</visual>
+		</gazebo>
+		<link name="link_6_y_rod">
+			<visual>
+				<origin rpy="-1.5708 0 0" xyz="0 0.1 0" />
+				<geometry>
+					<cylinder radius="0.005" length="0.2" /> </geometry>
+				<material name="green">
+					<color rgba="0.0 1.0 0.0 1.0" />
+				</material>
+			</visual>
+			<inertial>
+				<mass value="1e-5" />
+				<origin xyz="0 0 0" rpy="0 0 0" />
+				<inertia ixx="1e-6" ixy="0" ixz="0" iyy="1e-6" iyz="0" izz="1e-6" />
+			</inertial>
+		</link>
+		<joint name="link_6_y_rod_joint" type="fixed">
+			<parent link="link_6" />
+			<child link="link_6_y_rod" />
+			<origin xyz="0 0 0" rpy="0 0 0" />
+		</joint>
+		<gazebo reference="link_6_y_rod">
+			<visual>
+				<material>
+					<ambient>1 0 0 1</ambient>
+					<diffuse>1 0 0 1</diffuse>
+					<specular>0.1 0.1 0.1 1</specular>
+				</material>
+			</visual>
+		</gazebo>
+		<link name="link_6_x_rod">
+			<visual>
+				<origin rpy="0 1.5708 0" xyz="0.1 0 0" />
+				<geometry>
+					<cylinder radius="0.005" length="0.2" /> </geometry>
+				<material name="red">
+					<color rgba="1.0 0.0 0.0 1.0" />
+				</material>
+			</visual>
+			<inertial>
+				<mass value="1e-5" />
+				<origin xyz="0 0 0" rpy="0 0 0" />
+				<inertia ixx="1e-6" ixy="0" ixz="0" iyy="1e-6" iyz="0" izz="1e-6" />
+			</inertial>
+		</link>
+		<joint name="link_6_x_rod_joint" type="fixed">
+			<parent link="link_6" />
+			<child link="link_6_x_rod" />
+			<origin xyz="0 0 0" rpy="0 0 0" />
+		</joint>
+		<gazebo reference="link_6_x_rod">
+			<visual>
+				<material>
+					<ambient>1 0 0 1</ambient>
+					<diffuse>1 0 0 1</diffuse>
+					<specular>0.1 0.1 0.1 1</specular>
+				</material>
+			</visual>
+		</gazebo>
+		<!-- Camera -->
+		<link name="camera_link_optical"></link>
+		<joint name="camera_optical_joint" type="fixed">
+   			<parent link="link_6"/>
+    		<child link="camera_link_optical"/>
+    		<origin xyz="0 0 0" rpy="0 0 0"/>
+		</joint>
+		<gazebo reference="link_6">
+			<sensor name="camera_sensor" type="camera">
+				<pose>0.05 0 0.01 0 -1.5708 3.141519</pose>
+				<always_on>true</always_on>
+				<visualize>true</visualize>
+				<update_rate>30.0</update_rate>
+				<topic>/camera/image_raw</topic>
+				<gz_frame_id>camera_link_optical</gz_frame_id>
+				<camera name="camera">
+				<horizontal_fov>1.3962634</horizontal_fov>
+				<image>
+					<width>1280</width>
+					<height>720</height>
+					<format>R8G8B8</format>
+				</image>
+				<clip>
+					<near>0.02</near>
+					<far>300</far>
+				</clip>
+				</camera>
+			</sensor>
+		</gazebo>
     <xacro:dsr_transmission />
     <xacro:dsr_gazebo namespace="${namespace}" />

Commit message: add blower to mesh and xacro

File: dsr_description2/xacro/macro.m0609.white.xacro (robot description, xacro)
@@ -243,4 +243,31 @@
 			</visual>
 		</link>
+		<joint name="joint_fixed_attachment" type="fixed">
+      <parent link="link_6" />
+      <child link="blower_link" />
+      <origin rpy="0 0 0" xyz="0 0 0" />
+    </joint>
+    <link name="blower_link">
+			<collision>
+				<origin rpy="0 0 0" xyz="0 0 0.061" />
+				<geometry>
+					<cylinder radius="0.0625" length="0.122" />
+				</geometry>
+			</collision>
+			<visual>
+				<origin rpy="0 0 4.71238898038" xyz="0.006 0 -1.035" />
+				<geometry>
+					<mesh filename="package://dsr_description2/meshes/m0609_white/blower.stl" scale="0.001 0.001 0.001" />
+				</geometry>
+			</visual>
+      <inertial>
+        <mass value="0.1"/>
+        <origin xyz="0 0 0" rpy="0 0 0"/>
+        <inertia ixx="0.0001" ixy="0" ixz="0" iyy="0.0001" iyz="0" izz="0.0001"/>
+      </inertial>
+    </link>
+		<gazebo reference="blower_link">
+      <material>Gazebo/Blue</material>
+    </gazebo>
 		<!-- end effector axis for visualization-->
 		<link name="link_6_z_rod">

Commit message: fix robot arm blower mesh pose

File: dsr_description2/xacro/macro.m0609.white.xacro (robot description, xacro)
@@ -256,5 +256,5 @@
 			</collision>
 			<visual>
-				<origin rpy="0 0 4.71238898038" xyz="0.006 0 -1.035" />
+				<origin rpy="0 0 1.5707963267948966" xyz="-0.006 0 -1.035" />
 				<geometry>
 					<mesh filename="package://dsr_description2/meshes/m0609_white/blower.stl" scale="0.001 0.001 0.001" />

Commit message: enlarge blower collision mesh

File: dsr_description2/xacro/macro.m0609.white.xacro (robot description, xacro)
@@ -252,5 +252,5 @@
 				<origin rpy="0 0 0" xyz="0 0 0.061" />
 				<geometry>
-					<cylinder radius="0.0625" length="0.122" />
+					<cylinder radius="0.15" length="0.122" />
 				</geometry>
 			</collision>
